File: Pcb/Keyboard/Keyboard-Zerodeck/Keyboard-Zerodeck.kicad_pcb (KiCad board)
At the start: 2 copper layers, 220 x 90 mm, 80 parts, among them J1 SW_Push, K1 SW_Push, M1 SW_Push, P1 SW_Push, Q1 SW_Push, SW29 SW_Push, SW30 SW_Push, SW31 SW_Push, SW32 SW_Push, SW33 SW_Push, SW34 SW_Push, SW35 SW_Push, T1 SW_Push, U1 XIAO-RP2040-SMD, U2 MCP23017x-x-ML, U3 SW_Push, X1 SW_Push, Y1 SW_Push

Commit message: ain
Parts:
- removed ,1, .1, D38, SW29, SW30, SW31, SW32, SW33, SW34, SW35, Z1: SW_Push, Zero-Deck keys:Kailh_socket_PG1350
- removed D25, D36: 1N4148, Diode_THT:D_DO-35_SOD27_P7.62mm_Horizontal
- added Alt1: SW_Push, Zero-Deck keys:Kailh_socket_PG1350, F.Cu at (66.5, 108.5)
- added Comma1: SW_Push, Zero-Deck keys:Kailh_socket_PG1350, F.Cu at (156.5, 91.5)
- added Ctrl1: SW_Push, Zero-Deck keys:Kailh_socket_PG1350, F.Cu at (30.5, 108.5)
- added D39: 1N4148, Diode_SMD:D_SOD-123, F.Cu at (183.5, 91.3)
- added D40: 1N4148, Diode_SMD:D_SOD-123, F.Cu at (183.5, 74.5)
- added DICK1: SW_Push, Zero-Deck keys:Kailh_socket_PG1350, F.Cu at (66.5, 74.5)
- added Dot1: SW_Push, Zero-Deck keys:Kailh_socket_PG1350, F.Cu at (174.5, 91.5)
- added Function1: SW_Push, Zero-Deck keys:Kailh_socket_PG1350, F.Cu at (48.5, 108.5)
- added J2: Conn_01x05, Connector_JST:JST_PH_S5B-PH-K_1x05_P2.00mm_Horizontal, B.Cu at (194.0, 47.5)
- added J3: Conn_01x02, Connector_JST:JST_PH_S2B-PH-K_1x02_P2.00mm_Horizontal, B.Cu at (186.0, 47.5)
- added J4: Conn_01x02, Connector_JST:JST_PH_S2B-PH-K_1x02_P2.00mm_Horizontal, B.Cu at (208.0, 47.5)
- added MC1: SW_Push, Zero-Deck keys:Kailh_socket_PG1350, F.Cu at (156.5, 108.5)
- added MCC1: SW_Push, Zero-Deck keys:Kailh_socket_PG1350, F.Cu at (174.5, 108.5)
- added MCCC1: SW_Push, Zero-Deck keys:Kailh_socket_PG1350, F.Cu at (192.5, 108.5)
- added Space1: SW_Push, Zero-Deck keys:Kailh_socket_PG1350, F.Cu at (102.5, 108.5)
- added ZZZ1: SW_Push, Zero-Deck keys:Kailh_socket_PG1350, F.Cu at (30.5, 91.5)
- C1, R1, R2, R3, U1, U2: moved to F.Cu
- D1, D10, D11, D12, D13, D14, D15, D16, D17, D18, D19, D2, D20, D21, D22, D23, D24, D26, D27, D28, D29, D3, D30, D31, D32, D33, D34, D35, D37, D4, D5, D6, D7, D8, D9: footprint Diode_THT:D_DO-35_SOD27_P7.62mm_Horizontal -> Diode_SMD:D_SOD-123; moved to F.Cu
- moved D1 234.3 mm to (21.5, 57.6), turned to -90 degrees
- moved D29 217.3 mm to (21.5, 108.0), turned to -90 degrees
- moved D2 216.2 mm to (39.5, 57.6), turned to -90 degrees
- moved D30 199.1 mm to (39.5, 108.5), turned to -90 degrees
- moved D3 198.1 mm to (57.5, 57.5), turned to -90 degrees
- moved D13 189.1 mm to (57.5, 74.3), turned to -90 degrees
- moved D4 180.1 mm to (75.5, 57.5), turned to -90 degrees
- moved D14 170.8 mm to (75.5, 74.5), turned to -90 degrees
- moved D5 162.2 mm to (93.5, 57.5), turned to 90 degrees
- moved D15 152.5 mm to (93.5, 74.5), turned to 90 degrees
- moved D6 144.4 mm to (111.5, 57.5), turned to 90 degrees
- moved D16 134.2 mm to (111.5, 74.5), turned to 90 degrees
- moved D26 128.7 mm to (111.5, 91.5), turned to -90 degrees
- moved D7 126.8 mm to (129.5, 57.5), turned to 90 degrees
- moved D17 116.0 mm to (129.5, 74.7), turned to 90 degrees
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Connections:
- net /Col1 renamed /COL1
- net /Col2 renamed /COL2
- net /Col3 renamed /COL3
- net /Col4 renamed /COL4
- net /Col5 renamed /COL5
- net /R1 renamed /ROW1
- net /R2 renamed /ROW2
- net /R3 renamed /ROW3
- net /sck renamed /SCL
- C1 pad 1: /Gnd -> /GND
- D10 pad 1: /Col10 -> /COL10
- D16 pad 1: /Col6 -> /COL6
- D17 pad 1: /Col7 -> /COL7
- D18 pad 1: /Col8 -> /COL8
- D19 pad 1: /Col9 -> /COL9
- D26 pad 1: /Col7 -> /COL6
- D27 pad 1: /Col8 -> /COL7
- D28 pad 1: /Col9 -> /COL8
- D34 pad 1: /Col6 -> /COL6
- D35 pad 1: /Col7 -> /COL7
- D37 pad 1: /Col10 -> /COL9
- D6 pad 1: /Col6 -> /COL6
- D7 pad 1: /Col7 -> /COL7
- D8 pad 1: /Col8 -> /COL8
- D9 pad 1: /Col9 -> /COL9
- M1 pad 2: Net-(D26-A) -> Net-(D27-A)
- N1 pad 2: Net-(D25-A) -> Net-(D26-A)
- Shift1 pad 2: Net-(D37-A) -> Net-(D39-A)
- U1 pad 1: unconnected-(U1-D0-Pad1) -> /JOY_X
- U1 pad 13: unconnected-(U1-GND-Pad13) -> /GND
- U1 pad 18: unconnected-(U1-GND-Pad18) -> /GND
- U1 pad 2: unconnected-(U1-D1-Pad2) -> /JOY_Y
- U1 pad 20: /Gnd -> /GND
- U1 pad 3: unconnected-(U1-D2-Pad3) -> /JOY_SW
- U2 pad 1: /Col9 -> /COL9
- U2 pad 11: /Gnd -> /GND
- U2 pad 12: /Gnd -> /GND
- U2 pad 13: /Gnd -> /GND
- U2 pad 2: /Col10 -> /COL10
- U2 pad 20: /R4 -> /ROW4
- U2 pad 26: /Col6 -> /COL6
- U2 pad 27: /Col7 -> /COL7
- U2 pad 28: /Col8 -> /COL8
- U2 pad 3: unconnected-(U2-GPB6-Pad3) -> /JLEFT_CLICK
- U2 pad 4: unconnected-(U2-GPB7-Pad4) -> /JRIGHT_CLICK
- U2 pad 6: /Gnd -> /GND
