File: Pcb/Keyboard/Keyboard-Zerodeck/Keyboard-Zerodeck.kicad_sch (KiCad schematic)
At the start: 80 parts, among them J1 SW_Push, K1 SW_Push, M1 SW_Push, P1 SW_Push, Q1 SW_Push, SW29 SW_Push, SW30 SW_Push, SW31 SW_Push, SW32 SW_Push, SW33 SW_Push, SW34 SW_Push, SW35 SW_Push, T1 SW_Push, U1 XIAO-RP2040-SMD, U2 MCP23017x-x-ML, U3 SW_Push, X1 SW_Push, Y1 SW_Push

Commit message: ain
Parts:
- removed ,1, .1, A1, B1, C2, D38, E1, Enter1, F1, G1, H1, I1, J1, K1, L1, M1, N1, O1, P1, Q1, R4, S1, SW29, SW30, SW31, SW32, SW33, SW34, SW35, Shift1, T1, U3, V1, W1, X1, Y1, Z1: SW_Push, Zero-Deck keys:Kailh_socket_PG1350, symbol Switch:SW_Push
- removed D1, D10, D11, D12, D13, D14, D15, D16, D17, D18, D19, D2, D20, D21, D22, D23, D24, D25, D26, D27, D28, D29, D3, D30, D31, D32, D33, D34, D35, D36, D37, D4, D5, D6, D7, D8, D9: 1N4148, Diode_THT:D_DO-35_SOD27_P7.62mm_Horizontal, symbol Diode:1N4148
Connections:
- net Gnd is gone; now on net GND: C1.1, U1.20 (GND), U2.11 (A0), U2.12 (A1), U2.13 (A2), U2.6 (V_{SS})
- net JOY_X: now reaches U1.1 (D0)
- net GND: now reaches U1.13 (GND)
- net GND: now also U1.18 (GND)
- net JOY_Y: now reaches U1.2 (D1)
- net JOY_SW: now reaches U1.3 (D2)
- net JRIGHT_CLICK: now reaches U1.8 (D7)
- net JLEFT_CLICK: now reaches U1.9 (D8)
- net Col1 renamed COL1
- net Col10 renamed COL10
- net Col2 renamed COL2
- net Col3 renamed COL3
- net Col4 renamed COL4
- net Col5 renamed COL5
- net Col6 renamed COL6
- net Col7 renamed COL7
- net Col8 renamed COL8
- net Col9 renamed COL9
- net R1 renamed ROW1
- net R2 renamed ROW2
- net R3 renamed ROW3
- net R4 renamed ROW4
- net sck renamed SCL
- net sda renamed SDA
- no-connect marks 21 -> 12
Other:
- added sheet INTERCONNECTOR (INTERCONNECTOR.kicad_sch)
- added sheet JOYSTICK (JOYSTICK.kicad_sch)
- added sheet Key Matrix (Key_Matrix.kicad_sch)
- added sheet OLED_KEYBOARD (OLED_KEYBOARD.kicad_sch)
- note removed: "Col1"
- note removed: "Col2"
- note removed: "Col3"
- note removed: "Col4"
- note removed: "Col5"
- note removed: "Col6"
- note removed: "Col7"
- note removed: "Col8"
- note removed: "Col9"
- note removed: "Row1"
- note removed: "Row2"
- note removed: "Row3"
- moved on the sheet: C1, R1, R2, R3, U1, U2
